File: kicad/mboard-tall.kicad_pcb (KiCad board)
At the start: 2 copper layers, 50.8 x 25.4 mm, 14 parts

Commit message: pads and routes
Routing:
- net (no net): track 484.4 -> 484.9 mm
Changed lines of the file:
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@@
     (links 0)
     (no_connects 0)
-    (area 24.079999 34.239999 74.980001 59.740001)
+    (area 21.914524 32.403 76.157191 59.965001)
     (thickness 1.6)
     (drawings 9)
@@
   (page A4)
   (layers
-    (0 F.Cu signal)
+    (0 F.Cu signal hide)
     (31 B.Cu signal)
     (32 B.Adhes user hide)
@@
     (34 B.Paste user hide)
     (35 F.Paste user hide)
-    (36 B.SilkS user)
-    (37 F.SilkS user)
+    (36 B.SilkS user hide)
+    (37 F.SilkS user hide)
     (38 B.Mask user hide)
     (39 F.Mask user hide)
@@
       (drillshape 0)
       (scaleselection 1)
-      (outputdirectory /tmp/wthin))
+      (outputdirectory "C:/Users/Harry Potter/Documents/GitHub/protoh/oshpark/"))
   )
   (net 0 "")
@@
     (fp_line (start -8.89 -6.35) (end 11.43 -6.35) (layer F.SilkS) (width 0.15))
     (fp_line (start 11.43 -2.54) (end -8.89 -2.54) (layer F.SilkS) (width 0.15))
-    (pad 1 thru_hole rect (at -7.62 -5.08 90) (size 1.524 1.524) (drill 0.762) (layers *.Cu *.Mask F.SilkS))
-    (pad 2 thru_hole circle (at -5.08 -5.08 90) (size 1.524 1.524) (drill 0.762) (layers *.Cu *.Mask F.SilkS))
-    (pad 3 thru_hole circle (at -2.54 -5.08 90) (size 1.524 1.524) (drill 0.762) (layers *.Cu *.Mask F.SilkS))
-    (pad 4 thru_hole circle (at 0 -5.08 90) (size 1.524 1.524) (drill 0.762) (layers *.Cu *.Mask F.SilkS))
-    (pad 5 thru_hole circle (at 2.54 -5.08 90) (size 1.524 1.524) (drill 0.762) (layers *.Cu *.Mask F.SilkS))
-    (pad 6 thru_hole circle (at 5.08 -5.08 90) (size 1.524 1.524) (drill 0.762) (layers *.Cu *.Mask F.SilkS))
-    (pad 7 thru_hole circle (at 7.62 -5.08 90) (size 1.524 1.524) (drill 0.762) (layers *.Cu *.Mask F.SilkS))
-    (pad 8 thru_hole circle (at 10.16 -5.08 90) (size 1.524 1.524) (drill 0.762) (layers *.Cu *.Mask F.SilkS))
+    (pad VCC thru_hole rect (at -7.62 -5.08 180) (size 2.032 2.032) (drill 1.016) (layers *.Cu *.Mask F.SilkS))
+    (pad GND thru_hole circle (at -5.08 -5.08 90) (size 2.032 2.032) (drill 1.016) (layers *.Cu *.Mask F.SilkS))
+    (pad SCL thru_hole circle (at -2.54 -5.08 90) (size 2.032 2.032) (drill 1.016) (layers *.Cu *.Mask F.SilkS))
+    (pad SDA thru_hole circle (at 0 -5.08 90) (size 2.032 2.032) (drill 1.016) (layers *.Cu *.Mask F.SilkS))
+    (pad XCL thru_hole circle (at 2.54 -5.08 90) (size 2.032 2.032) (drill 1.016) (layers *.Cu *.Mask F.SilkS))
+    (pad XDA thru_hole circle (at 5.08 -5.08 90) (size 2.032 2.032) (drill 1.016) (layers *.Cu *.Mask F.SilkS))
+    (pad ADD thru_hole circle (at 7.62 -5.08 90) (size 2.032 2.032) (drill 1.016) (layers *.Cu *.Mask F.SilkS))
+    (pad INI thru_hole circle (at 10.16 -5.08 90) (size 2.032 2.032) (drill 1.016) (layers *.Cu *.Mask F.SilkS))
   )
   (module LEDs:LED-3MM (layer F.Cu)
@@
   (segment (start 41.402 38.608) (end 29.21 38.608) (width 0.25) (layer B.Cu) (net 0))
   (segment (start 29.21 38.608) (end 27.686 37.084) (width 0.25) (layer B.Cu) (net 0))
-  (segment (start 59.69 41.656) (end 57.15 41.656) (width 0.25) (layer B.Cu) (net 0))
+  (segment (start 59.69 41.91) (end 57.15 41.91) (width 0.25) (layer B.Cu) (net 0))
   (segment (start 54.61 38.354) (end 55.88 37.084) (width 0.25) (layer B.Cu) (net 0))
-  (segment (start 54.61 41.656) (end 54.61 38.354) (width 0.25) (layer B.Cu) (net 0))
-  (segment (start 57.15 41.656) (end 54.61 41.656) (width 0.25) (layer B.Cu) (net 0))
+  (segment (start 54.61 41.91) (end 54.61 38.354) (width 0.25) (layer B.Cu) (net 0))
+  (segment (start 57.15 41.91) (end 54.61 41.91) (width 0.25) (layer B.Cu) (net 0))
   (segment (start 55.88 37.084) (end 55.88 36.83) (width 0.25) (layer B.Cu) (net 0))
   (segment (start 72.898 40.64) (end 65.786 40.64) (width 0.25) (layer B.Cu) (net 0))
@@
   (segment (start 66.294 38.608) (end 66.04 38.354) (width 0.25) (layer B.Cu) (net 0))
   (segment (start 59.69 38.608) (end 66.294 38.608) (width 0.25) (layer B.Cu) (net 0))
-  (segment (start 59.69 41.656) (end 59.69 38.608) (width 0.25) (layer B.Cu) (net 0))
-  (segment (start 65.532 41.656) (end 59.69 41.656) (width 0.25) (layer B.Cu) (net 0))
-  (segment (start 65.532 40.894) (end 65.532 41.656) (width 0.25) (layer B.Cu) (net 0))
+  (segment (start 59.69 41.91) (end 59.69 38.608) (width 0.25) (layer B.Cu) (net 0))
+  (segment (start 65.532 41.91) (end 59.69 41.91) (width 0.25) (layer B.Cu) (net 0))
+  (segment (start 65.532 40.894) (end 65.532 41.91) (width 0.25) (layer B.Cu) (net 0))
   (segment (start 65.786 40.64) (end 65.532 40.894) (width 0.25) (layer B.Cu) (net 0))
   (segment (start 53.34 38.862) (end 63.5 38.862) (width 0.25) (layer F.Cu) (net 0))
@@
   (segment (start 34.29 46.99) (end 36.83 46.99) (width 0.25) (layer F.Cu) (net 0) (status 10))
   (segment (start 36.83 48.26) (end 38.1 48.26) (width 0.25) (layer F.Cu) (net 0) (status 20))
-  (segment (start 40.64 54.356) (end 33.02 54.356) (width 0.25) (layer F.Cu) (net 0))
-  (segment (start 33.02 54.356) (end 33.02 55.88) (width 0.25) (layer F.Cu) (net 0) (status 20))
-  (segment (start 40.64 53.34) (end 40.64 54.356) (width 0.25) (layer F.Cu) (net 0) (status 10))
-  (segment (start 38.1 44.704) (end 41.91 44.704) (width 0.25) (layer F.Cu) (net 0))
-  (segment (start 41.91 44.704) (end 41.91 57.15) (width 0.25) (layer F.Cu) (net 0))
+  (segment (start 39.37 54.61) (end 33.02 54.61) (width 0.25) (layer F.Cu) (net 0))
+  (segment (start 33.02 54.61) (end 33.02 55.88) (width 0.25) (layer F.Cu) (net 0) (status 800020))
+  (segment (start 40.64 53.34) (end 39.37 54.61) (width 0.25) (layer F.Cu) (net 0) (status 400010))
+  (segment (start 38.1 44.45) (end 41.91 44.45) (width 0.25) (layer F.Cu) (net 0))
+  (segment (start 41.91 44.45) (end 41.91 57.15) (width 0.25) (layer F.Cu) (net 0))
   (segment (start 41.91 57.15) (end 35.56 57.15) (width 0.25) (layer F.Cu) (net 0))
   (segment (start 35.56 57.15) (end 35.56 55.88) (width 0.25) (layer F.Cu) (net 0) (status 20))
-  (segment (start 38.1 45.72) (end 38.1 44.704) (width 0.25) (layer F.Cu) (net 0) (status 10))
-  (segment (start 39.624 51.816) (end 39.624 54.356) (width 0.25) (layer B.Cu) (net 0))
-  (segment (start 39.624 54.356) (end 38.1 55.88) (width 0.25) (layer B.Cu) (net 0) (status 20))
-  (segment (start 40.64 50.8) (end 39.624 51.816) (width 0.25) (layer B.Cu) (net 0) (status 10))
+  (segment (start 38.1 45.72) (end 38.1 44.45) (width 0.25) (layer F.Cu) (net 0) (status 400010))
+  (segment (start 39.37 51.816) (end 39.37 54.356) (width 0.25) (layer B.Cu) (net 0))
+  (segment (start 39.37 54.356) (end 38.1 55.88) (width 0.25) (layer B.Cu) (net 0) (status 800020))
+  (segment (start 40.64 50.8) (end 39.37 51.816) (width 0.25) (layer B.Cu) (net 0) (status 400010))
 )

Commit message: larger 5v holes. Flight Computer.
Routing:
- net (no net): track 484.9 -> 483.4 mm
Other:
- board text added: "Flight Computer"

Commit message: ESP8266 and 3V fixes
Parts:
- moved LDO33 5.08 mm to (34.3, 52.1), turned to 180 degrees
Routing:
- net (no net): track 483.4 -> 449.4 mm
Other:
- board text added: "PlugCopter 2015-May donpark.org"
- board text removed: "PlugCopter 2015-Apr donpark.org"

Commit message: add sonar plugs
Parts:
- added REF**: Pin_Header_Straight_1x04, Pin_Headers:Pin_Header_Straight_1x04, F.Cu at (43.4, 59.4)
- added REF**: Pin_Header_Straight_1x04, Pin_Headers:Pin_Header_Straight_1x04, F.Cu at (54.1, 59.4)
- moved REF** 2.27 mm to (72.4, 58.9), turned to 0 degrees
Routing:
- net (no net): track 449.4 -> 497.2 mm
Other:
- board size 50.8 x 25.4 mm -> 50.8 x 26.4 mm
- board text added: "Flight"
- board text removed: "Flight Computer"

Commit message: size tweaks
Parts:
- REF: renamed from REF**; value LED-D -> LEDD
- S1: renamed from REF**; value Pin_Header_Straight_1x04 -> (none)
- renumbered REF** to S2
Changed lines of the file:
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@@
     (links 0)
     (no_connects 0)
-    (area 21.914524 32.403 76.157191 59.965001)
+    (area 21.914524 32.403 75.823953 61.411001)
     (thickness 1.6)
     (drawings 14)
@@
     (34 B.Paste user hide)
     (35 F.Paste user hide)
-    (36 B.SilkS user hide)
+    (36 B.SilkS user)
     (37 F.SilkS user)
     (38 B.Mask user hide)
@@
     (descr "LED 3mm - Lead pitch 100mil (2,54mm)")
     (tags "LED led 3mm 3MM 100mil 2,54mm")
-    (fp_text reference REF** (at 1.778 -2.794) (layer F.SilkS) hide
-      (effects (font (size 1 1) (thickness 0.15)))
-    )
-    (fp_text value LED-D (at 5 0) (layer F.SilkS)
+    (fp_text reference REF (at 1.778 -2.794) (layer F.SilkS) hide
+      (effects (font (size 1 1) (thickness 0.15)))
+    )
+    (fp_text value LEDD (at 0.682 -2.54) (layer F.SilkS)
       (effects (font (size 1 1) (thickness 0.15)))
     )
@@
     (descr "Through hole pin header")
     (tags "pin header")
-    (fp_text reference REF** (at 0 -5.1 90) (layer F.SilkS)
-      (effects (font (size 1 1) (thickness 0.15)))
-    )
-    (fp_text value Pin_Header_Straight_1x04 (at 0 -3.1 90) (layer F.Fab)
+    (fp_text reference S1 (at 0 -2.56 90) (layer F.SilkS)
+      (effects (font (size 1 1) (thickness 0.15)))
+    )
+    (fp_text value "" (at 0 -3.1 90) (layer F.Fab) hide
       (effects (font (size 1 1) (thickness 0.15)))
     )
@@
     (descr "Through hole pin header")
     (tags "pin header")
-    (fp_text reference REF** (at 0 -5.1 90) (layer F.SilkS)
-      (effects (font (size 1 1) (thickness 0.15)))
-    )
-    (fp_text value Pin_Header_Straight_1x04 (at 0 -3.1 90) (layer F.Fab)
+    (fp_text reference S2 (at 0 8.91 90) (layer F.SilkS)
+      (effects (font (size 1 1) (thickness 0.15)))
+    )
+    (fp_text value Pin_Header_Straight_1x04 (at 0 -3.1 90) (layer F.Fab) hide
       (effects (font (size 1 1) (thickness 0.15)))
     )
@@
   (gr_line (start 74.93 34.29) (end 74.93 59.69) (angle 90) (layer Edge.Cuts) (width 0.1))
   (gr_line (start 24.13 34.29) (end 74.93 34.29) (angle 90) (layer Edge.Cuts) (width 0.1))
-  (segment (start 59.182 59.436) (end 59.182 56.642) (width 0.25) (layer F.Cu) (net 0) (status 400000))
-  (segment (start 59.182 56.642) (end 58.42 55.88) (width 0.25) (layer F.Cu) (net 0) (status 800000))
-  (segment (start 56.642 59.436) (end 56.642 56.642) (width 0.25) (layer F.Cu) (net 0) (status 400000))
-  (segment (start 56.642 56.642) (end 55.88 55.88) (width 0.25) (layer F.Cu) (net 0) (status 800000))
-  (segment (start 62.23 52.07) (end 62.23 58.928) (width 0.25) (layer B.Cu) (net 0) (status 800000))
-  (segment (start 62.23 58.928) (end 61.722 59.436) (width 0.25) (layer B.Cu) (net 0) (status C00000))
-  (segment (start 54.61 54.61) (end 54.61 58.928) (width 0.25) (layer F.Cu) (net 0) (status 800000))
-  (segment (start 54.61 58.928) (end 54.102 59.436) (width 0.25) (layer F.Cu) (net 0) (status C00000))
+  (segment (start 59.182 59.436) (end 59.182 56.642) (width 0.25) (layer F.Cu) (net 0))
+  (segment (start 59.182 56.642) (end 58.42 55.88) (width 0.25) (layer F.Cu) (net 0))
+  (segment (start 56.642 59.436) (end 56.642 56.642) (width 0.25) (layer F.Cu) (net 0))
+  (segment (start 56.642 56.642) (end 55.88 55.88) (width 0.25) (layer F.Cu) (net 0))
+  (segment (start 62.23 52.07) (end 62.23 58.928) (width 0.25) (layer B.Cu) (net 0))
+  (segment (start 62.23 58.928) (end 61.722 59.436) (width 0.25) (layer B.Cu) (net 0))
+  (segment (start 54.61 54.61) (end 54.61 58.928) (width 0.25) (layer F.Cu) (net 0))
+  (segment (start 54.61 58.928) (end 54.102 59.436) (width 0.25) (layer F.Cu) (net 0))
   (segment (start 48.514 59.436) (end 48.514 58.674) (width 0.25) (layer F.Cu) (net 0))
   (segment (start 48.514 58.674) (end 45.72 55.88) (width 0.25) (layer F.Cu) (net 0))
